Commit message: update models with correct rod plates

File: urdf_srdf/updated_mass/2x10kg/urdf/_centauro_robot.urdf (robot description, URDF)
Before this commit: robot centauro, 58 links, 57 joints
Links:
- removed link ball1
- removed link ball1_tip
- removed link ball2
- removed link ball2_tip
- added link rod_plate1, mass 10.01; collision mesh filename=package://centauro_urdf/meshes/simple/RodPlate.stl scale=0.001 -0.001 0.001; visual mesh filename=package://centauro_urdf/meshes/simple/RodPlate.stl scale=0.001 -0.001 0.001
- added link rod_plate1_tip
- added link rod_plate2, mass 10.01; collision mesh filename=package://centauro_urdf/meshes/simple/RodPlate.stl scale=0.001 0.001 0.001; visual mesh filename=package://centauro_urdf/meshes/simple/RodPlate.stl scale=0.001 0.001 0.001
- added link rod_plate2_tip
Joints:
- removed joint j_ball1_fixed
- removed joint j_ball1_tip
- removed joint j_ball2_fixed
- removed joint j_ball2_tip
- added joint j_rod_plate1_fixed: type fixed, parent rod_plate1, child arm1_8
- added joint j_rod_plate1_tip: type fixed, parent rod_plate1, child rod_plate1_tip, origin xyz=0.06 0.0 -0.16 rpy=0.0 0.0 0.349066
- added joint j_rod_plate2_fixed: type fixed, parent rod_plate2, child arm2_8
- added joint j_rod_plate2_tip: type fixed, parent rod_plate2, child rod_plate2_tip, origin xyz=0.06 0.0 -0.16 rpy=0.0 0.0 -0.349066
- joint j_arm1_8: child ball1 -> rod_plate1
- joint j_arm2_8: child ball2 -> rod_plate2

File: urdf_srdf/updated_mass/2x10kg/urdf/centauro.urdf (robot description, URDF)
Before this commit: robot centauro, 58 links, 57 joints
Links:
- removed link ball1
- removed link ball1_tip
- removed link ball2
- removed link ball2_tip
- added link rod_plate1, mass 10.01; collision mesh filename=package://centauro_urdf/meshes/simple/RodPlate.stl scale=0.001 -0.001 0.001; visual mesh filename=package://centauro_urdf/meshes/simple/RodPlate.stl scale=0.001 -0.001 0.001
- added link rod_plate1_tip
- added link rod_plate2, mass 10.01; collision mesh filename=package://centauro_urdf/meshes/simple/RodPlate.stl scale=0.001 0.001 0.001; visual mesh filename=package://centauro_urdf/meshes/simple/RodPlate.stl scale=0.001 0.001 0.001
- added link rod_plate2_tip
Joints:
- removed joint j_ball1_fixed
- removed joint j_ball1_tip
- removed joint j_ball2_fixed
- removed joint j_ball2_tip
- added joint j_rod_plate1_fixed: type fixed, parent rod_plate1, child arm1_8
- added joint j_rod_plate1_tip: type fixed, parent rod_plate1, child rod_plate1_tip, origin xyz=0.06 0.0 -0.16 rpy=0.0 0.0 0.349066
- added joint j_rod_plate2_fixed: type fixed, parent rod_plate2, child arm2_8
- added joint j_rod_plate2_tip: type fixed, parent rod_plate2, child rod_plate2_tip, origin xyz=0.06 0.0 -0.16 rpy=0.0 0.0 -0.349066
- joint j_arm1_8: child ball1 -> rod_plate1
- joint j_arm2_8: child ball2 -> rod_plate2

File: urdf_srdf/updated_mass/2x10kg/urdf/centauro_base.urdf.xacro (robot description, xacro)
@@ -45,10 +45,19 @@
 	<xacro:if value="${ADD_BALL_END_EFFECTOR}">
 		<xacro:include filename="parts/ball.urdf.xacro" />
-		<xacro:ball_end_effector arm_num="1"  parent_link="arm1_7">
+		<xacro:ball_end_effector arm_num="1"  parent_link="arm1_7" ball_mass="1.27">
       			<origin xyz="0. 0. 0." rpy="0. 0. 0."/>
    		</xacro:ball_end_effector>
-		<xacro:ball_end_effector arm_num="2"  parent_link="arm2_7">
+		<xacro:ball_end_effector arm_num="2"  parent_link="arm2_7" ball_mass="1.27">
       			<origin xyz="0. 0. 0." rpy="0. 0. 0."/>
    		</xacro:ball_end_effector>
+	</xacro:if>
+	<xacro:if value="${ADD_ROD_PLATE_END_EFFECTOR}">
+		<xacro:include filename="parts/rod_plate.urdf.xacro" />
+		<xacro:rod_plate_end_effector arm_num="1" rot="1" parent_link="arm1_7" rod_mass="10.01">
+      			<origin xyz="0. 0. 0." rpy="0. 0. 0."/>
+   		</xacro:rod_plate_end_effector>
+		<xacro:rod_plate_end_effector arm_num="2" rot="-1"  parent_link="arm2_7" rod_mass="10.01">
+      			<origin xyz="0. 0. 0." rpy="0. 0. 0."/>
+   		</xacro:rod_plate_end_effector>
 	</xacro:if>
 	<xacro:include filename="parts/head.urdf.xacro" />

File: urdf_srdf/updated_mass/2x10kg/urdf/centauro_virtual_frame.urdf (robot description, URDF)
Before this commit: robot centauro, 64 links, 63 joints
Links:
- removed link ball1
- removed link ball1_tip
- removed link ball2
- removed link ball2_tip
- added link rod_plate1, mass 10.01; collision mesh filename=package://centauro_urdf/meshes/simple/RodPlate.stl scale=0.001 -0.001 0.001; visual mesh filename=package://centauro_urdf/meshes/simple/RodPlate.stl scale=0.001 -0.001 0.001
- added link rod_plate1_tip
- added link rod_plate2, mass 10.01; collision mesh filename=package://centauro_urdf/meshes/simple/RodPlate.stl scale=0.001 0.001 0.001; visual mesh filename=package://centauro_urdf/meshes/simple/RodPlate.stl scale=0.001 0.001 0.001
- added link rod_plate2_tip
Joints:
- removed joint j_ball1_fixed
- removed joint j_ball1_tip
- removed joint j_ball2_fixed
- removed joint j_ball2_tip
- added joint j_rod_plate1_fixed: type fixed, parent rod_plate1, child arm1_8
- added joint j_rod_plate1_tip: type fixed, parent rod_plate1, child rod_plate1_tip, origin xyz=0.06 0.0 -0.16 rpy=0.0 0.0 0.349066
- added joint j_rod_plate2_fixed: type fixed, parent rod_plate2, child arm2_8
- added joint j_rod_plate2_tip: type fixed, parent rod_plate2, child rod_plate2_tip, origin xyz=0.06 0.0 -0.16 rpy=0.0 0.0 -0.349066
- joint j_arm1_8: child ball1 -> rod_plate1
- joint j_arm2_8: child ball2 -> rod_plate2

File: urdf_srdf/updated_mass/2x10kg/urdf/centauro_virtual_frame_robot.urdf (robot description, URDF)
Before this commit: robot centauro, 64 links, 63 joints
Links:
- removed link ball1
- removed link ball1_tip
- removed link ball2
- removed link ball2_tip
- added link rod_plate1, mass 10.01; collision mesh filename=package://centauro_urdf/meshes/simple/RodPlate.stl scale=0.001 -0.001 0.001; visual mesh filename=package://centauro_urdf/meshes/simple/RodPlate.stl scale=0.001 -0.001 0.001
- added link rod_plate1_tip
- added link rod_plate2, mass 10.01; collision mesh filename=package://centauro_urdf/meshes/simple/RodPlate.stl scale=0.001 0.001 0.001; visual mesh filename=package://centauro_urdf/meshes/simple/RodPlate.stl scale=0.001 0.001 0.001
- added link rod_plate2_tip
Joints:
- removed joint j_ball1_fixed
- removed joint j_ball1_tip
- removed joint j_ball2_fixed
- removed joint j_ball2_tip
- added joint j_rod_plate1_fixed: type fixed, parent rod_plate1, child arm1_8
- added joint j_rod_plate1_tip: type fixed, parent rod_plate1, child rod_plate1_tip, origin xyz=0.06 0.0 -0.16 rpy=0.0 0.0 0.349066
- added joint j_rod_plate2_fixed: type fixed, parent rod_plate2, child arm2_8
- added joint j_rod_plate2_tip: type fixed, parent rod_plate2, child rod_plate2_tip, origin xyz=0.06 0.0 -0.16 rpy=0.0 0.0 -0.349066
- joint j_arm1_8: child ball1 -> rod_plate1
- joint j_arm2_8: child ball2 -> rod_plate2

File: urdf_srdf/updated_mass/2x5kg/urdf/_centauro_robot.urdf (robot description, URDF)
Before this commit: robot centauro, 58 links, 57 joints
Links:
- removed link ball1
- removed link ball1_tip
- removed link ball2
- removed link ball2_tip
- added link rod_plate1, mass 5.01; collision mesh filename=package://centauro_urdf/meshes/simple/RodPlate.stl scale=0.001 -0.001 0.001; visual mesh filename=package://centauro_urdf/meshes/simple/RodPlate.stl scale=0.001 -0.001 0.001
- added link rod_plate1_tip
- added link rod_plate2, mass 5.01; collision mesh filename=package://centauro_urdf/meshes/simple/RodPlate.stl scale=0.001 0.001 0.001; visual mesh filename=package://centauro_urdf/meshes/simple/RodPlate.stl scale=0.001 0.001 0.001
- added link rod_plate2_tip
Joints:
- removed joint j_ball1_fixed
- removed joint j_ball1_tip
- removed joint j_ball2_fixed
- removed joint j_ball2_tip
- added joint j_rod_plate1_fixed: type fixed, parent rod_plate1, child arm1_8
- added joint j_rod_plate1_tip: type fixed, parent rod_plate1, child rod_plate1_tip, origin xyz=0.06 0.0 -0.16 rpy=0.0 0.0 0.349066
- added joint j_rod_plate2_fixed: type fixed, parent rod_plate2, child arm2_8
- added joint j_rod_plate2_tip: type fixed, parent rod_plate2, child rod_plate2_tip, origin xyz=0.06 0.0 -0.16 rpy=0.0 0.0 -0.349066
- joint j_arm1_8: child ball1 -> rod_plate1
- joint j_arm2_8: child ball2 -> rod_plate2

File: urdf_srdf/updated_mass/2x5kg/urdf/centauro.urdf (robot description, URDF)
Before this commit: robot centauro, 58 links, 57 joints
Links:
- removed link ball1
- removed link ball1_tip
- removed link ball2
- removed link ball2_tip
- added link rod_plate1, mass 5.01; collision mesh filename=package://centauro_urdf/meshes/simple/RodPlate.stl scale=0.001 -0.001 0.001; visual mesh filename=package://centauro_urdf/meshes/simple/RodPlate.stl scale=0.001 -0.001 0.001
- added link rod_plate1_tip
- added link rod_plate2, mass 5.01; collision mesh filename=package://centauro_urdf/meshes/simple/RodPlate.stl scale=0.001 0.001 0.001; visual mesh filename=package://centauro_urdf/meshes/simple/RodPlate.stl scale=0.001 0.001 0.001
- added link rod_plate2_tip
Joints:
- removed joint j_ball1_fixed
- removed joint j_ball1_tip
- removed joint j_ball2_fixed
- removed joint j_ball2_tip
- added joint j_rod_plate1_fixed: type fixed, parent rod_plate1, child arm1_8
- added joint j_rod_plate1_tip: type fixed, parent rod_plate1, child rod_plate1_tip, origin xyz=0.06 0.0 -0.16 rpy=0.0 0.0 0.349066
- added joint j_rod_plate2_fixed: type fixed, parent rod_plate2, child arm2_8
- added joint j_rod_plate2_tip: type fixed, parent rod_plate2, child rod_plate2_tip, origin xyz=0.06 0.0 -0.16 rpy=0.0 0.0 -0.349066
- joint j_arm1_8: child ball1 -> rod_plate1
- joint j_arm2_8: child ball2 -> rod_plate2

File: urdf_srdf/updated_mass/2x5kg/urdf/centauro_base.urdf.xacro (robot description, xacro)
@@ -45,10 +45,19 @@
 	<xacro:if value="${ADD_BALL_END_EFFECTOR}">
 		<xacro:include filename="parts/ball.urdf.xacro" />
-		<xacro:ball_end_effector arm_num="1"  parent_link="arm1_7">
+		<xacro:ball_end_effector arm_num="1"  parent_link="arm1_7" ball_mass="1.27">
       			<origin xyz="0. 0. 0." rpy="0. 0. 0."/>
    		</xacro:ball_end_effector>
-		<xacro:ball_end_effector arm_num="2"  parent_link="arm2_7">
+		<xacro:ball_end_effector arm_num="2"  parent_link="arm2_7" ball_mass="1.27">
       			<origin xyz="0. 0. 0." rpy="0. 0. 0."/>
    		</xacro:ball_end_effector>
+	</xacro:if>
+	<xacro:if value="${ADD_ROD_PLATE_END_EFFECTOR}">
+		<xacro:include filename="parts/rod_plate.urdf.xacro" />
+		<xacro:rod_plate_end_effector arm_num="1" rot="1" parent_link="arm1_7" rod_mass="5.01">
+      			<origin xyz="0. 0. 0." rpy="0. 0. 0."/>
+   		</xacro:rod_plate_end_effector>
+		<xacro:rod_plate_end_effector arm_num="2" rot="-1"  parent_link="arm2_7" rod_mass="5.01">
+      			<origin xyz="0. 0. 0." rpy="0. 0. 0."/>
+   		</xacro:rod_plate_end_effector>
 	</xacro:if>
 	<xacro:include filename="parts/head.urdf.xacro" />

File: urdf_srdf/updated_mass/2x5kg/urdf/centauro_virtual_frame.urdf (robot description, URDF)
Before this commit: robot centauro, 64 links, 63 joints
Links:
- removed link ball1
- removed link ball1_tip
- removed link ball2
- removed link ball2_tip
- added link rod_plate1, mass 5.01; collision mesh filename=package://centauro_urdf/meshes/simple/RodPlate.stl scale=0.001 -0.001 0.001; visual mesh filename=package://centauro_urdf/meshes/simple/RodPlate.stl scale=0.001 -0.001 0.001
- added link rod_plate1_tip
- added link rod_plate2, mass 5.01; collision mesh filename=package://centauro_urdf/meshes/simple/RodPlate.stl scale=0.001 0.001 0.001; visual mesh filename=package://centauro_urdf/meshes/simple/RodPlate.stl scale=0.001 0.001 0.001
- added link rod_plate2_tip
Joints:
- removed joint j_ball1_fixed
- removed joint j_ball1_tip
- removed joint j_ball2_fixed
- removed joint j_ball2_tip
- added joint j_rod_plate1_fixed: type fixed, parent rod_plate1, child arm1_8
- added joint j_rod_plate1_tip: type fixed, parent rod_plate1, child rod_plate1_tip, origin xyz=0.06 0.0 -0.16 rpy=0.0 0.0 0.349066
- added joint j_rod_plate2_fixed: type fixed, parent rod_plate2, child arm2_8
- added joint j_rod_plate2_tip: type fixed, parent rod_plate2, child rod_plate2_tip, origin xyz=0.06 0.0 -0.16 rpy=0.0 0.0 -0.349066
- joint j_arm1_8: child ball1 -> rod_plate1
- joint j_arm2_8: child ball2 -> rod_plate2

File: urdf_srdf/updated_mass/2x5kg/urdf/centauro_virtual_frame_robot.urdf (robot description, URDF)
Before this commit: robot centauro, 64 links, 63 joints
Links:
- removed link ball1
- removed link ball1_tip
- removed link ball2
- removed link ball2_tip
- added link rod_plate1, mass 5.01; collision mesh filename=package://centauro_urdf/meshes/simple/RodPlate.stl scale=0.001 -0.001 0.001; visual mesh filename=package://centauro_urdf/meshes/simple/RodPlate.stl scale=0.001 -0.001 0.001
- added link rod_plate1_tip
- added link rod_plate2, mass 5.01; collision mesh filename=package://centauro_urdf/meshes/simple/RodPlate.stl scale=0.001 0.001 0.001; visual mesh filename=package://centauro_urdf/meshes/simple/RodPlate.stl scale=0.001 0.001 0.001
- added link rod_plate2_tip
Joints:
- removed joint j_ball1_fixed
- removed joint j_ball1_tip
- removed joint j_ball2_fixed
- removed joint j_ball2_tip
- added joint j_rod_plate1_fixed: type fixed, parent rod_plate1, child arm1_8
- added joint j_rod_plate1_tip: type fixed, parent rod_plate1, child rod_plate1_tip, origin xyz=0.06 0.0 -0.16 rpy=0.0 0.0 0.349066
- added joint j_rod_plate2_fixed: type fixed, parent rod_plate2, child arm2_8
- added joint j_rod_plate2_tip: type fixed, parent rod_plate2, child rod_plate2_tip, origin xyz=0.06 0.0 -0.16 rpy=0.0 0.0 -0.349066
- joint j_arm1_8: child ball1 -> rod_plate1
- joint j_arm2_8: child ball2 -> rod_plate2

File: urdf_srdf/updated_mass/2x5kg/urdf/gazebo/materials.gazebo.xacro (robot description, xacro)
@@ -67,4 +67,12 @@
 </gazebo>
 </xacro:if>
+<xacro:if value="${ADD_ROD_PLATE_END_EFFECTOR}">
+<gazebo reference="rod_plate1">
+	<material>Gazebo/BlueTransparent</material>
+</gazebo>
+<gazebo reference="rod_plate2">
+	<material>Gazebo/GreenTransparent</material>
+</gazebo>
+</xacro:if>
 </xacro:if>
 </robot>

File: urdf_srdf/updated_mass/2x5kg/urdf/parts/ball.urdf.xacro (robot description, xacro)
@@ -1,9 +1,9 @@
 <?xml version="1.0"?>
 <robot xmlns:xacro="http://ros.org/wiki/xacro">
-<xacro:macro name="ball_end_effector" params="arm_num parent_link *origin">
+<xacro:macro name="ball_end_effector" params="arm_num parent_link ball_mass *origin">
 <link name="ball${arm_num}">
     <inertial>
       <origin xyz="${-1.0072498e-02*mmTom} ${3.7590658e-02*mmTom} ${1.9772332e+01*mmTom}" rpy="0 0 0"/>
-      <mass value="5.0"/>
+      <mass value="${ball_mass}"/>
       <inertia ixx="${2.3061092e+03*mm2Tom2}"  ixy="${2.9181758e-01*mm2Tom2}"  ixz="${-2.1246684e-01*mm2Tom2}" iyy="${2.3053155e+03*mm2Tom2}" iyz="${7.9290978e-01*mm2Tom2}" izz="${3.0675616e+03*mm2Tom2}" />
     </inertial>
