Commit message: correct wheel_mot gain in saved urdfs, adapt scripts to paper plots

File: urdf_srdf/updated_mass/0+10kg/urdf/gazebo/xbot.gazebo.xacro (robot description, xacro)
@@ -16,8 +16,8 @@
             <gain name="medium_mot" p="1000" d="10"/>
             <gain name="big_mot"    p="3000" d="10"/>
-            <gain name="wheel_mot"  p="0" d="10"/>
+            <gain name="wheel_mot"  p="250" d="10"/>
             <pid name="neck_yaw" profile="lowpwr_mot"/>
             <pid name="neck_pitch" profile="lowpwr_mot"/>
-            <pid name="neck_velodyne" p="250"  d="20"/>
+            <pid name="neck_velodyne" p="0"  d="20"/>
             <pid name="j_arm1_1" profile="medium_mot"/>
             <pid name="j_arm1_2" profile="medium_mot"/>

File: urdf_srdf/updated_mass/2x10kg/urdf/gazebo/materials.gazebo.xacro (robot description, xacro)
@@ -69,8 +69,8 @@
 <xacro:if value="${ADD_ROD_PLATE_END_EFFECTOR}">
 <gazebo reference="rod_plate1">
-	<material>Gazebo/BlueTransparent</material>
+	<material>Gazebo/GreyTransparent</material>
 </gazebo>
 <gazebo reference="rod_plate2">
-	<material>Gazebo/GreenTransparent</material>
+	<material>Gazebo/GreyTransparent</material>
 </gazebo>
 </xacro:if>
