Commit message: updated rod plate urdf 2x10kg and removed the rest, added argument for arm ee in centauro_payload_world.launch

File: urdf_srdf/rod_plates/2x10kg/urdf/_centauro_robot.urdf (robot description, URDF)
Before this commit: robot centauro, 58 links, 57 joints
Joints:
- joint j_rod_plate1_fixed: origin (none) -> xyz=0.048407693 -0.020035723 -0.077533287 rpy=0 0 0
- joint j_rod_plate2_fixed: origin (none) -> xyz=0.048407693 0.020035723 -0.077533287 rpy=0 0 0

File: urdf_srdf/rod_plates/2x10kg/urdf/centauro.urdf (robot description, URDF)
Before this commit: robot centauro, 58 links, 57 joints
Joints:
- joint j_rod_plate1_fixed: origin (none) -> xyz=0.048407693 -0.020035723 -0.077533287 rpy=0 0 0
- joint j_rod_plate2_fixed: origin (none) -> xyz=0.048407693 0.020035723 -0.077533287 rpy=0 0 0

File: urdf_srdf/rod_plates/2x10kg/urdf/centauro_base.urdf.xacro (robot description, xacro)
@@ -45,8 +45,8 @@
 	<xacro:if value="${ADD_BALL_END_EFFECTOR}">
 		<xacro:include filename="parts/ball.urdf.xacro" />
-		<xacro:ball_end_effector arm_num="1"  parent_link="arm1_7" ball_mass="1.27">
+		<xacro:ball_end_effector arm_num="1"  parent_link="arm1_7" ball_mass="0.27">
       			<origin xyz="0. 0. 0." rpy="0. 0. 0."/>
    		</xacro:ball_end_effector>
-		<xacro:ball_end_effector arm_num="2"  parent_link="arm2_7" ball_mass="1.27">
+		<xacro:ball_end_effector arm_num="2"  parent_link="arm2_7" ball_mass="0.27">
       			<origin xyz="0. 0. 0." rpy="0. 0. 0."/>
    		</xacro:ball_end_effector>

File: urdf_srdf/rod_plates/2x10kg/urdf/centauro_virtual_frame.urdf (robot description, URDF)
Before this commit: robot centauro, 64 links, 63 joints
Joints:
- joint j_rod_plate1_fixed: origin (none) -> xyz=0.048407693 -0.020035723 -0.077533287 rpy=0 0 0
- joint j_rod_plate2_fixed: origin (none) -> xyz=0.048407693 0.020035723 -0.077533287 rpy=0 0 0

File: urdf_srdf/rod_plates/2x10kg/urdf/centauro_virtual_frame_robot.urdf (robot description, URDF)
Before this commit: robot centauro, 64 links, 63 joints
Joints:
- joint j_rod_plate1_fixed: origin (none) -> xyz=0.048407693 -0.020035723 -0.077533287 rpy=0 0 0
- joint j_rod_plate2_fixed: origin (none) -> xyz=0.048407693 0.020035723 -0.077533287 rpy=0 0 0

File: urdf_srdf/rod_plates/2x10kg/urdf/gazebo/materials.gazebo.xacro (robot description, xacro)
@@ -69,8 +69,8 @@
 <xacro:if value="${ADD_ROD_PLATE_END_EFFECTOR}">
 <gazebo reference="rod_plate1">
-	<material>Gazebo/GreyTransparent</material>
+	<material>Gazebo/BlueTransparent</material>
 </gazebo>
 <gazebo reference="rod_plate2">
-	<material>Gazebo/GreyTransparent</material>
+	<material>Gazebo/GreenTransparent</material>
 </gazebo>
 </xacro:if>
