Commit message: updated friction of saved urdf 2x10 with ballhands, added bashfiles for 3 locomotion only and other stepups

File: urdf_srdf/ball_hand/2x10kg/urdf/gazebo/centauro.gazebo.xacro (robot description, xacro)
@@ -1,4 +1,5 @@
 <?xml version="1.0"?>
 <robot xmlns:xacro="http://ros.org/wiki/xacro">
+<xacro:property name="friction_coeff" value="0.9" />
 <xacro:if value="${ADD_LEGS}">
 <gazebo reference="wheel_1">
@@ -8,10 +9,10 @@
             <friction>
                 <ode>
-                    <mu>1.0</mu>
-                    <mu2>1.0</mu2>
-                </ode>
-                <bullet>
-                    <friction>1.0</friction>
-                    <friction2>1.0</friction2>
+                    <mu>${friction_coeff}</mu>
+                    <mu2>${friction_coeff}</mu2>
+                </ode>
+                <bullet>
+                    <friction>${friction_coeff}</friction>
+                    <friction2>${friction_coeff}</friction2>
                 </bullet>
             </friction>
@@ -38,10 +39,10 @@
             <friction>
                 <ode>
-                    <mu>1.0</mu>
-                    <mu2>1.0</mu2>
-                </ode>
-                <bullet>
-                    <friction>1.0</friction>
-                    <friction2>1.0</friction2>
+                    <mu>${friction_coeff}</mu>
+                    <mu2>${friction_coeff}</mu2>
+                </ode>
+                <bullet>
+                    <friction>${friction_coeff}</friction>
+                    <friction2>${friction_coeff}</friction2>
                 </bullet>
             </friction>
@@ -68,10 +69,10 @@
             <friction>
                 <ode>
-                    <mu>1.0</mu>
-                    <mu2>1.0</mu2>
-                </ode>
-                <bullet>
-                    <friction>1.0</friction>
-                    <friction2>1.0</friction2>
+                    <mu>${friction_coeff}</mu>
+                    <mu2>${friction_coeff}</mu2>
+                </ode>
+                <bullet>
+                    <friction>${friction_coeff}</friction>
+                    <friction2>${friction_coeff}</friction2>
                 </bullet>
             </friction>
@@ -98,10 +99,10 @@
             <friction>
                 <ode>
-                    <mu>1.0</mu>
-                    <mu2>1.0</mu2>
-                </ode>
-                <bullet>
-                    <friction>1.0</friction>
-                    <friction2>1.0</friction2>
+                    <mu>${friction_coeff}</mu>
+                    <mu2>${friction_coeff}</mu2>
+                </ode>
+                <bullet>
+                    <friction>${friction_coeff}</friction>
+                    <friction2>${friction_coeff}</friction2>
                 </bullet>
             </friction>
